File: eagle/alpha/rev02/rev02.sch (EAGLE design)
At the start: 322 parts, among them CN1 HOST, IC1 IS45S32160F, IC3 N25Q128A13ES, Q3 2N7002, Q5 ASFL1, Q6 2N7002, T1 BC847, T2 BC847, T3 BC818, U1 MC14551BDG, U2 MC74HC1G14DTT1G, U3 ATTINY828R-AU, U4 MC14551BDG, U5 23K640-I/SN, U6 MCP79412-I/SN, U7 XC7A200TFBG484, Y1 12 MHz

Commit message: connect first SDRAM, add USB MGMT UART.
Parts:
- added C10, C180, C182, C183, C185, C187, C188, C189, C197, C200, C201, C9: 0.1 uF, resistor:C-EUC0402
- added C11, C12: 5 pF, rcl:C-EUC0603
- added C179, C181: 4.7 uF, resistor:C-EUC0603
- added C184, C186: 10 uF, resistor:C-EUC0805
- added C194, C195, C196, C198, C199, C206, C207, C208: 0.1uF, resistor:C-EUC0402
- added CN2: HOST, adafruit:USBMINIB
- added FB3, FB4: 600R 500mA, microbuilder:FERRITE_0603MP
- added LED17: YELLOW, SparkFun-LED:LED0603
- added LED18: GREEN, SparkFun-LED:LED0603
- added R69: 10K, resistor:R-EU_R0402
- added R70: 12K, resistor:R-EU_R0402
- added R71, R72: 220, resistor:R-EU_R0402
- added U$10: FT232H_SERIAL, FT232H:FT232H_SERIAL
- added Y2: 12 MHz, microbuilder:CRYSTALTHIN
Connections:
- removed net FPGA_FMC_CLK: U$1G$4.PD3/FMC_CLK, U7B13.IO_L12P_T1_MRCC_13
- new net FMC_CLK: IC1.CLK, U$1G$4.PD3/FMC_CLK, U7B13.IO_L12P_T1_MRCC_13
- new net FMC_NBL0: IC1.DQM0, U$1G$4.FMC_NBL0/PE0
- new net FMC_NBL1: IC1.DQM1, U$1G$4.FMC_NBL1/PE1
- new net FMC_NBL2: IC1.DQM2, U$1G$4.FMC_NBL2/PI4
- new net FMC_NBL3: IC1.DQM3, U$1G$4.FMC_NBL3/PI5
- new net FMC_SDCKE0: IC1.CKE, U$1G$1.FMC_SDCKE0/PC3
- new net FMC_SDNCAS: IC1.!CAS, U$1G$4.FMC_SDNCAS/PG15
- new net FMC_SDNE0: IC1.!CS, U$1G$1.FMC_SDNE0/PC2
- new net FMC_SDNRAS: IC1.!RAS, U$1G$2.PF11/FMC_SDNRAS
- new net FMC_SDNWE: IC1.!WE, U$1G$1.FMC_SDNWE/PC0
- new net FT_MGMT_CTS: U$10.CTS#
- new net FT_MGMT_DTR: U$10.DTR#
- new net FT_MGMT_RTS: U$10.RTS#
- new net FT_MGMT_RXD: U$10.RXD
- new net FT_MGMT_TXD: U$10.TXD
- new net FT_MGMT_VCC3V3: C181.1, C182.1, C187.1, C188.1, C189.1, FB3.P$1, FB4.P$1, LED17.A, LED18.A, R69.2, U$10.VCCD, U$10.VCCIO@12, U$10.VCCIO@24, U$10.VCCIO@46
- new net FT_MGMT_VPHY: U$10.VPHY
- new net FT_MGMT_VPLL: C185.1, C186.1, FB3.P$2, U$10.VPLL
- new net FT_MGMT_VREGIN: C179.1, C180.1, CN2.VBUS, U$10.VREGIN
- new net FT_REF1: R70.1, U$10.REF
- new net FT_RESET1: R69.1, U$10.!RESET
- new net FT_RXLED1: R71.2, U$10.RXLED#
- new net FT_TXLED1: R72.2, U$10.TXLED#
- new net FT_VCCA1: C9.1, U$10.VCCA
- new net FT_VCCORE1: C10.1, U$10.VCCORE
- new net N$6: LED17.C, R71.1
- new net N$7: LED18.C, R72.1
- new net N$8: C11.2, U$10.XCSO, Y2.2
- new net N$9: C12.2, U$10.XCSI, Y2.1
- new net USB_MGMT_DM: CN2.D-, U$10.DM
- new net USB_MGMT_DP: CN2.D+, U$10.DP
- net FMC_A0: now also IC1.A0
- net FMC_A1: now also IC1.A1
- net FMC_A10: now also IC1.A10
- net FMC_A11: now also IC1.A11
- net FMC_A12: now also IC1.A12
- net FMC_A14: now also IC1.BA0
- net FMC_A15: now also IC1.BA1
- net FMC_A2: now also IC1.A2
- net FMC_A22: now also U$1G$1.PE6/FMC_A22
- net FMC_A23: now also U$1G$1.PE2/FMC_A23
- net FMC_A24: now also U$1G$4.PG13/FMC_A24
- net FMC_A25: now also U$1G$4.PG14/FMC_A25
- net FMC_A3: now also IC1.A3
- net FMC_A4: now also IC1.A4
- net FMC_A5: now also IC1.A5
- net FMC_A6: now also IC1.A6
- net FMC_A7: now also IC1.A7
- net FMC_A8: now also IC1.A8
- net FMC_A9: now also IC1.A9
- net FMC_D10: now also IC1.DQ9
- net FMC_D18: no longer IC1.DQ19
- net FMC_D19: now also IC1.DQ19
- net FMC_D9: no longer IC1.DQ9
- net FT_VPHY: now also C183.1, C184.1, FB4.P$2
- net GND: now also C10.2, C11.1, C12.1, C179.2, C180.2, C181.2, C182.2, C183.2, C184.2, C185.2, C186.2, C187.2, C188.2, C189.2, C194.2, C195.2, C196.2, C197.2, C198.2, C199.2, C200.2, C201.2, C206.2, C207.2, C208.2, C9.2, CN2.GND, IC1.VSS@44, IC1.VSS@58, IC1.VSS@72, IC1.VSS@86, IC1.VSSQ@12, IC1.VSSQ@32, IC1.VSSQ@38, IC1.VSSQ@46, IC1.VSSQ@52, IC1.VSSQ@6, IC1.VSSQ@78, IC1.VSSQ@84, R70.2, U$10.AGND@4, U$10.AGND@41, U$10.AGND@9, U$10.GND@10, U$10.GND@11, U$10.GND@22, U$10.GND@23, U$10.GND@35, U$10.GND@36, U$10.GND@47, U$10.GND@48, U$10.TEST
- net VCCO_3V3: now also C194.1, C195.1, C196.1, C197.1, C198.1, C199.1, C200.1, C201.1, C206.1, C207.1, C208.1, IC1.VDD@15, IC1.VDD@29, IC1.VDD@43, IC1.VDDQ@35, IC1.VDDQ@41, IC1.VDDQ@49, IC1.VDDQ@55, IC1.VDDQ@75, IC1.VDDQ@81
Other:
- note added: "Analog switch to boot FPGA from config memory, or from ARM XXX this probably needs more HW support. FPGA is SPI master when booting from config memory, but should be SPI slave when being fed a bitstream from the ARM."
- note added: "To mitigate component ageing in the avalanche noise circuit, this jumper can be used to decide if FPGA/ARM/None should be allowed to turn off the entropy source (default On through pull-up)"
- note added: "XXX add circuitry to allow FPGA/ARM to control sinking of the 18V from the 10K pull-up on pin 2."
- note added: "XXX this shared for all FMC?"
- note added: "XXX with the addition of the two SDRAM chips, do we need an CKE signal to the FPGA?"
- note removed: "Analog switch to boot FPGA from config memory, or from ARM"
- note removed: "Jumper deciding if FPGA/ARM/None should be allowed to turn off the entropy source (default On through pull-up)"

Commit message: updates after todays call with Pavel
Parts:
- added C190, C191, C192, C202, C203, C209, C210, C211: 0.1uF, resistor:C-EUC0402
- added C193, C204, C205: 0.1 uF, resistor:C-EUC0402
- added C212: 0.1 uF, resistor:C-EUC0603
- added C213: 2.2 uF LowESR, resistor:C-EUC0603
- added IC2: IS45S32160F, Alpha-IC:IS45S32160F
- added IC4: N25Q128A13ES, altera-configdevices:N25Q128A13ES
- added Q1: 2N7002, transistors_gaui:2N7002
- added R73, R74: 4.7k, resistor:R-EU_R0603
- added R75: 10K, resistor:R-EU_R0402
- added R76: 1K, resistor:R-EU_R0402
- JP2: device SparkFun-Connectors:M03LOCK -> jumper:JP1Q
Connections:
- removed net FPGA_ENTROPY_ENABLE: JP2.1
- removed net FPGA_PROM_CS_N: IC3.!S, R9.1, U1.X0
- new net FMC_SDCKE1: IC2.CKE, U$1G$4.FMC_SDCKE1/PB5
- new net FMC_SDCLK: IC1.CLK, IC2.CLK, U$1G$3.FMC_SDCLK/PG8
- new net FMC_SDNE1: IC2.!CS, U$1G$4.FMC_SDNE1/PB6
- new net FPGA_ENTROPY_DISABLE: R76.1, U7B16.IO_L11N_T1_SRCC_16
- new net KSM_PROM_CS_N: IC3.!S, IC4.!S, R73.2, R9.1, U1.X0
- new net KSM_PROM_MISO: IC4.DQ1, U$1G$2.PA6/SPI1_MISO
- new net KSM_PROM_MOSI: IC4.DQ0, U$1G$2.PA7/SPI1_MOSI
- new net KSM_PROM_SCLK: IC4.C, U$1G$2.PA5/SPI1_SCK
- new net N$11: Q1.G, R75.1, R76.2
- new net N$14: JP2.2, Q1.D
- net 15V_LDO_ENABLE: now also JP2.1; no longer JP2.2
- net FMC_A0: now also IC2.A0
- net FMC_A1: now also IC2.A1
- net FMC_A10: now also IC2.A10
- net FMC_A11: now also IC2.A11
- net FMC_A12: now also IC2.A12
- net FMC_A14: now also IC2.BA0
- net FMC_A15: now also IC2.BA1
- net FMC_A2: now also IC2.A2
- net FMC_A3: now also IC2.A3
- net FMC_A4: now also IC2.A4
- net FMC_A5: now also IC2.A5
- net FMC_A6: now also IC2.A6
- net FMC_A7: now also IC2.A7
- net FMC_A8: now also IC2.A8
- net FMC_A9: now also IC2.A9
- net FMC_CLK: no longer IC1.CLK
- net FMC_D0: now also IC2.DQ0
- net FMC_D1: now also IC2.DQ1
- net FMC_D10: now also IC2.DQ10, IC2.DQ9
- net FMC_D11: now also IC2.DQ11
- net FMC_D12: now also IC2.DQ12
- net FMC_D13: now also IC2.DQ13
- net FMC_D14: now also IC2.DQ14
- net FMC_D15: now also IC2.DQ15
- net FMC_D16: now also IC2.DQ16
- net FMC_D17: now also IC2.DQ17
- net FMC_D18: now also IC2.DQ18
- net FMC_D19: now also IC2.DQ19
- net FMC_D2: now also IC2.DQ2
- net FMC_D20: now also IC2.DQ20
- net FMC_D21: now also IC2.DQ21
- net FMC_D22: now also IC2.DQ22
- net FMC_D23: now also IC2.DQ23
- net FMC_D24: now also IC2.DQ24
- net FMC_D25: now also IC2.DQ25
- net FMC_D26: now also IC2.DQ26
- net FMC_D27: now also IC2.DQ27
- net FMC_D28: now also IC2.DQ28
- net FMC_D29: now also IC2.DQ29
- net FMC_D3: now also IC2.DQ3
- net FMC_D30: now also IC2.DQ30
- net FMC_D31: now also IC2.DQ31
- net FMC_D4: now also IC2.DQ4
- net FMC_D5: now also IC2.DQ5
- net FMC_D6: now also IC2.DQ6
- net FMC_D7: now also IC2.DQ7
- net FMC_D8: now also IC2.DQ8
- net FMC_NBL0: now also IC2.DQM0
- net FMC_NBL1: now also IC2.DQM1
- net FMC_NBL2: now also IC2.DQM2
- net FMC_NBL3: now also IC2.DQM3
- net FMC_SDNCAS: now also IC2.!CAS
- net FMC_SDNRAS: now also IC2.!RAS
- net FMC_SDNWE: now also IC2.!WE
- net GND: now also C190.2, C191.2, C192.2, C193.2, C202.2, C203.2, C204.2, C205.2, C209.2, C210.2, C211.2, C212.2, C213.2, IC2.VSS@44, IC2.VSS@58, IC2.VSS@72, IC2.VSS@86, IC2.VSSQ@12, IC2.VSSQ@32, IC2.VSSQ@38, IC2.VSSQ@46, IC2.VSSQ@52, IC2.VSSQ@6, IC2.VSSQ@78, IC2.VSSQ@84, IC4.VSS, Q1.S, R73.1, R74.1, R75.2
- net PWR_18V: now also C213.1
- net VCCO_3V3: now also C190.1, C191.1, C192.1, C193.1, C202.1, C203.1, C204.1, C205.1, C209.1, C210.1, C211.1, C212.1, IC1.VDD@1, IC1.VDDQ@3, IC2.VDD@1, IC2.VDD@15, IC2.VDD@29, IC2.VDD@43, IC2.VDDQ@3, IC2.VDDQ@35, IC2.VDDQ@41, IC2.VDDQ@49, IC2.VDDQ@55, IC2.VDDQ@75, IC2.VDDQ@81, IC4.!HOLD!/DQ3, IC4.!W!/VPP/DQ2, IC4.VCC, R74.2
Other:
- note added: "*) HOLD feature not used"
- note added: "FPGA_GPIO_B* is blue LEDs in Alpha block diagram. Suggest pin header instead for more versatility."
- note added: "Keystore memory This memory holds cryptographic keys wrapped with master key in MKM."
- note added: "Look at Novena"
- note added: "Management access USB UART"
- note added: "XXX EEPROM for USB settings or not?"
- note added: "XXX check with Joachim if it is enough that STM32 can rewrite FPGA config memory"
- note removed: "Another identical SRAM chip goes here"
- note removed: "Keystore memory (>= 8 MByte) goes here"
- note removed: "THESE TWO TO AT TINY"
- note removed: "XXX add circuitry to allow FPGA/ARM to control sinking of the 18V from the 10K pull-up on pin 2."
- note removed: "XXX this shared for all FMC?"
- note removed: "XXX with the addition of the two SDRAM chips, do we need an CKE signal to the FPGA?"
- moved on the sheet: C194, C195, C196, C197, C198, C199, C200, C201, C206, C207, C208, IC1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
